Commit message: end of camera

File: robot_urdf/urdf/robot4.xacro (robot description, xacro)
@@ -117,81 +117,81 @@
   <!--arm definition -->
   <link name="arm_base_link">
-  	<inertial>
-  		<mass value="0.1"/>
-  		<origin xyz="0 0 0" rpy="0 0 0" />
-  		<inertia ixx="0.0000416666667" ixy="0" ixz="0" iyy="0.0000416666667" iyz="0" izz="0.0000416666667"/>
-  	</inertial>
-  	<collision>
-  	  <origin xyz="0 0 0" rpy="0 0 0"/>
+    <inertial>
+      <mass value="0.1"/>
+      <origin xyz="0 0 0" rpy="0 0 0"/>
+      <inertia ixx="0.0000416666667" ixy="0" ixz="0" iyy="0.0000416666667" iyz="0" izz="0.0000416666667"/>
+    </inertial>
+    <collision>
+      <origin xyz="0 0 0" rpy="0 0 0"/>
       <geometry>
-        <box size="0.1 0.1 0.1"/>
+        <box size="0.1 0.1 0.06"/>
       </geometry>
-  	</collision>
-  	<visual>
-  	  <origin xyz="0 0 0" rpy="0 0 0"/>
+    </collision>
+    <visual>
+      <origin xyz="0 0 0" rpy="0 0 0"/>
       <geometry>
-        <box size="0.1 0.1 0.1"/>
+        <box size="0.1 0.1 0.05"/>
       </geometry>
-      <material name="red" />
-  	</visual>
+      <material name="red"/>
+    </visual>
   </link>
   <joint name="arm_base_to_base" type="fixed">
-  	<origin rpy="0 0 0" xyz="0 0 0.085"/>
-  	<parent link="link_chassis"/>
-  	<child link="arm_base_link"/>
+    <origin rpy="0 0 0" xyz="0 0 0.055"/>
+    <parent link="link_chassis"/>
+    <child link="arm_base_link"/>
   </joint>
   <link name="arm_link_01">
-  	<inertial>
-  		<mass value="0.025"/>
-  		<origin xyz="0 0 0" rpy="0 0 0" />
-  		<inertia ixx="0.000010279" ixy="0" ixz="0" iyy="0.000010279" iyz="0" izz="0.000007225"/>
-  	</inertial>
-  	<collision>
-  	  <origin xyz="0 0 0" rpy="0 0 0"/>
+    <inertial>
+      <mass value="0.025"/>
+      <origin xyz="0 0 0" rpy="0 0 0"/>
+      <inertia ixx="0.000010279" ixy="0" ixz="0" iyy="0.000010279" iyz="0" izz="0.000007225"/>
+    </inertial>
+    <collision>
+      <origin xyz="0 0 0" rpy="0 0 0"/>
       <geometry>
-        <cylinder radius="0.04" length="0.08"/>
+        <cylinder radius="0.04" length="0.15"/>
       </geometry>
-  	</collision>
-  	<visual>
-  	  <origin xyz="0 0 0" rpy="0 0 0"/>
+    </collision>
+    <visual>
+      <origin xyz="0 0 0" rpy="0 0 0"/>
       <geometry>
-        <cylinder radius="0.04" length="0.08"/>
+        <cylinder radius="0.04" length="0.15"/>
       </geometry>
-      <material name="red" />
-  	</visual>
+      <material name="red"/>
+    </visual>
   </link>
   <joint name="arm_joint_01" type="continuous">
-  	<axis xyz="0 0 1"/>
-  	<origin rpy="0 0 0" xyz="0 0 0.09"/>
-  	<parent link="arm_base_link"/>
-  	<child link="arm_link_01"/>
+    <axis xyz="0 0 1"/>
+    <origin rpy="0 0 0" xyz="0 0 0.05"/>
+    <parent link="arm_base_link"/>
+    <child link="arm_link_01"/>
   </joint>
   <link name="camera_link">
-	    <collision>
-	      <origin xyz="0 0 0.06" rpy="0 0 0"/>
-	      <geometry>
-		<box size="0.05 0.05 0.05"/>
-	      </geometry>
-	    </collision>
-	    <visual>
-	      <origin xyz="0 0 0.06" rpy="0 0 0"/>
-	      <geometry>
-		<box size="0.05 0.05 0.05"/>
-	      </geometry>
-	      <material name="red">
-		<color rgba="1 0 0 1"/>
-	      </material>
-	    </visual>
-	    <inertial>
-	      <mass value="1e-5" />
-	      <origin xyz="0 0 0" rpy="0 0 0"/>
-	      <inertia ixx="1e-6" ixy="0" ixz="0" iyy="1e-6" iyz="0" izz="1e-6" />
-	    </inertial>
+    <collision>
+      <origin xyz="0 0 0.04" rpy="0 0 0"/>
+      <geometry>
+        <box size="0.05 0.05 0.05"/>
+      </geometry>
+    </collision>
+    <visual>
+      <origin xyz="0 0 0.06" rpy="0 0 0"/>
+      <geometry>
+        <box size="0.05 0.05 0.05"/>
+      </geometry>
+      <material name="red">
+        <color rgba="1 0 0 1"/>
+      </material>
+    </visual>
+    <inertial>
+      <mass value="1e-5"/>
+      <origin xyz="0 0 0" rpy="0 0 0"/>
+      <inertia ixx="1e-6" ixy="0" ixz="0" iyy="1e-6" iyz="0" izz="1e-6"/>
+    </inertial>
   </link>
   <joint name="camera_joint" type="fixed">
-	    <axis xyz="0 0 1" />
-	    <origin xyz="0.0 0 0.0" rpy="0 0 0"/>
-	    <parent link="arm_link_01"/>
-	    <child link="camera_link"/>
-	 </joint>
+    <axis xyz="0 1 0"/>
+    <origin xyz="0 0 0.04" rpy="0 0 0"/>
+    <parent link="arm_link_01"/>
+    <child link="camera_link"/>
+  </joint>
 </robot>
