Commit message: pddl part

File: rob_nav/urdf/robot_nav.xacro (robot description, xacro)
@@ -1,5 +1,5 @@
 <?xml version="1.0"?>
-<robot xmlns:xacro="http://www.ros.org/wiki/xacro" name="robot_xacro">
- <xacro:include filename="$(find rob_nav)/urdf/robot.gazebo"/>
+<robot xmlns:xacro="http://www.ros.org/wiki/xacro" name="robot_nav_xacro">
+ <xacro:include filename="$(find rob_nav)/urdf/robot_nav.gazebo"/>
  <xacro:include filename="$(find rob_nav)/urdf/materials.xacro" />
   <!-- Inertia definition (cylinder, wheel + chassis) -->
@@ -92,58 +92,4 @@
   <xacro:joint_wheel name="joint_right_wheel"  child="link_right_wheel"  origin_xyz="-0.05 0.15 0"  />
   <xacro:joint_wheel name="joint_left_wheel"   child="link_left_wheel"   origin_xyz="-0.05 -0.15 0"  />
-  <!--arm definition -->
-  <!--
-  <link name="arm_base_link">
-  	<inertial>
-  		<mass value="0.1"/>
-  		<origin xyz="0 0 0" rpy="0 0 0" />
-  		<inertia ixx="0.0000416666667" ixy="0" ixz="0" iyy="0.0000416666667" iyz="0" izz="0.0000416666667"/>
-  	</inertial>
-  	<collision>
-  	  <origin xyz="0 0 0" rpy="0 0 0"/>
-      <geometry>
-        <box size="0.1 0.1 0.06"/>
-      </geometry>
-  	</collision>
-  	<visual>
-  	  <origin xyz="0 0 0" rpy="0 0 0"/>
-      <geometry>
-        <box size="0.1 0.1 0.05"/>
-      </geometry>
-      <material name="red" />
-  	</visual>
-  </link>
-  <joint name="arm_base_to_base" type="fixed">
-  	<origin rpy="0 0 0" xyz="0 0 0.055"/>
-  	<parent link="link_chassis"/>
-  	<child link="arm_base_link"/>
-  </joint>
-  <link name="arm_link_01">
-  	<inertial>
-  		<mass value="0.025"/>
-  		<origin xyz="0 0 0" rpy="0 0 0" />
-  		<inertia ixx="0.000010279" ixy="0" ixz="0" iyy="0.000010279" iyz="0" izz="0.000007225"/>
-  	</inertial>
-  	<collision>
-  	  <origin xyz="0 0 0" rpy="0 0 0"/>
-      <geometry>
-        <cylinder radius="0.04" length="0.15"/>
-      </geometry>
-  	</collision>
-  	<visual>
-  	  <origin xyz="0 0 0" rpy="0 0 0"/>
-      <geometry>
-        <cylinder radius="0.04" length="0.15"/>
-      </geometry>
-      <material name="red" />
-  	</visual>
-  </link>
-  <joint name="arm_joint_01" type="continuous">
-  	<axis xyz="0 0 1"/>
-  	<origin rpy="0 0 0" xyz="0 0 0.05"/>
-  	<parent link="arm_base_link"/>
-  	<child link="arm_link_01"/>
-  </joint>
-   -->
   <!-- Camera -->
   <link name="camera_link">
@@ -171,5 +117,5 @@
   <joint name="camera_joint" type="fixed">
     <axis xyz="0 1 0"/>
-    <origin xyz="0.23 0 0.235" rpy="0 0 0"/>
+    <origin xyz="0.23 0 0.0 " rpy="0 0 0"/>
     <parent link="link_chassis"/>
     <child link="camera_link"/>
